File: KiCad/StateMachineTest/8BitLED.sch (KiCad schematic (older format))
At the start: 18 parts, among them U8 74HC245

Commit message: ERC OK
Changed lines of the file:
@@
 $Descr A4 11693 8268
 encoding utf-8
-Sheet 7 58
+Sheet 41 58
 Title ""
 Date ""
@@
 Wire Wire Line
 	4500 3450 4500 3550
-Text HLabel 3450 2000 0    50   Input ~ 0
-VAL[0..7]
 $Comp
 L power:GND #PWR0130
@@
 AR Path="/60E33DBC/5F767EF5/5F82FFCD/5F315EF7" Ref="C125"  Part="1"
 AR Path="/60E33DBC/5F768DA1/5F82FFCD/5F315EF7" Ref="C130"  Part="1"
-F 0 "C19" V 4421 1800 50  0000 C CNN
+F 0 "C115" V 4421 1800 50  0000 C CNN
 F 1 "0u1" V 4512 1800 50  0000 C CNN
 F 2 "Capacitor_SMD:C_0603_1608Metric" H 4650 1800 50  0001 C CNN
@@
 AR Path="/60E33DBC/5F767EF5/5F82FFCD/5F5B8923" Ref="R100"  Part="1"
 AR Path="/60E33DBC/5F768DA1/5F82FFCD/5F5B8923" Ref="R108"  Part="1"
-F 0 "R11" V 5350 2300 50  0000 C CNN
+F 0 "R84" V 5350 2300 50  0000 C CNN
 F 1 "rled" V 5350 2000 50  0000 C CNN
 F 2 "Resistor_SMD:R_0603_1608Metric" H 5400 2150 50  0001 C CNN
@@
 AR Path="/60E33DBC/5F767EF5/5F82FFCD/5F5BB79D" Ref="R101"  Part="1"
 AR Path="/60E33DBC/5F768DA1/5F82FFCD/5F5BB79D" Ref="R109"  Part="1"
-F 0 "R12" V 5350 2400 50  0000 C CNN
+F 0 "R85" V 5350 2400 50  0000 C CNN
 F 1 "rled" V 5350 2100 50  0000 C CNN
 F 2 "Resistor_SMD:R_0603_1608Metric" H 5400 2250 50  0001 C CNN
@@
 AR Path="/60E33DBC/5F767EF5/5F82FFCD/5F5BBC63" Ref="R102"  Part="1"
 AR Path="/60E33DBC/5F768DA1/5F82FFCD/5F5BBC63" Ref="R110"  Part="1"
-F 0 "R13" V 5350 2500 50  0000 C CNN
+F 0 "R86" V 5350 2500 50  0000 C CNN
 F 1 "rled" V 5350 2200 50  0000 C CNN
 F 2 "Resistor_SMD:R_0603_1608Metric" H 5400 2350 50  0001 C CNN
@@
 AR Path="/60E33DBC/5F767EF5/5F82FFCD/5F5BC15A" Ref="R103"  Part="1"
 AR Path="/60E33DBC/5F768DA1/5F82FFCD/5F5BC15A" Ref="R111"  Part="1"
-F 0 "R14" V 5350 2600 50  0000 C CNN
+F 0 "R87" V 5350 2600 50  0000 C CNN
 F 1 "rled" V 5350 2300 50  0000 C CNN
 F 2 "Resistor_SMD:R_0603_1608Metric" H 5400 2450 50  0001 C CNN
@@
 AR Path="/60E33DBC/5F767EF5/5F82FFCD/5F5BC5A8" Ref="R104"  Part="1"
 AR Path="/60E33DBC/5F768DA1/5F82FFCD/5F5BC5A8" Ref="R112"  Part="1"
-F 0 "R15" V 5350 2700 50  0000 C CNN
+F 0 "R88" V 5350 2700 50  0000 C CNN
 F 1 "rled" V 5350 2400 50  0000 C CNN
 F 2 "Resistor_SMD:R_0603_1608Metric" H 5400 2550 50  0001 C CNN
@@
 AR Path="/60E33DBC/5F767EF5/5F82FFCD/5F5BCA40" Ref="R105"  Part="1"
 AR Path="/60E33DBC/5F768DA1/5F82FFCD/5F5BCA40" Ref="R113"  Part="1"
-F 0 "R16" V 5350 2800 50  0000 C CNN
+F 0 "R89" V 5350 2800 50  0000 C CNN
 F 1 "rled" V 5350 2500 50  0000 C CNN
 F 2 "Resistor_SMD:R_0603_1608Metric" H 5400 2650 50  0001 C CNN
@@
 AR Path="/60E33DBC/5F767EF5/5F82FFCD/5F5BDE32" Ref="R106"  Part="1"
 AR Path="/60E33DBC/5F768DA1/5F82FFCD/5F5BDE32" Ref="R114"  Part="1"
-F 0 "R17" V 5350 2900 50  0000 C CNN
+F 0 "R90" V 5350 2900 50  0000 C CNN
 F 1 "rled" V 5350 2600 50  0000 C CNN
 F 2 "Resistor_SMD:R_0603_1608Metric" H 5400 2750 50  0001 C CNN
@@
 AR Path="/60E33DBC/5F767EF5/5F82FFCD/5F5BE2E1" Ref="R107"  Part="1"
 AR Path="/60E33DBC/5F768DA1/5F82FFCD/5F5BE2E1" Ref="R115"  Part="1"
-F 0 "R18" V 5350 3000 50  0000 C CNN
+F 0 "R91" V 5350 3000 50  0000 C CNN
 F 1 "rled" V 5350 2700 50  0000 C CNN
 F 2 "Resistor_SMD:R_0603_1608Metric" H 5400 2850 50  0001 C CNN
@@
 AR Path="/60E33DBC/5F767EF5/5F82FFCD/5F5C179E" Ref="D86"  Part="1"
 AR Path="/60E33DBC/5F768DA1/5F82FFCD/5F5C179E" Ref="D94"  Part="1"
-F 0 "D11" H 5700 2100 50  0000 C CNN
+F 0 "D70" H 5700 2100 50  0000 C CNN
 F 1 "LED" H 6000 2100 50  0000 C CNN
 F 2 "LED_SMD:LED_0805_2012Metric" V 5900 2150 50  0001 C CNN
@@
 AR Path="/60E33DBC/5F767EF5/5F82FFCD/5F5C2BC5" Ref="D90"  Part="1"
 AR Path="/60E33DBC/5F768DA1/5F82FFCD/5F5C2BC5" Ref="D98"  Part="1"
-F 0 "D15" H 5900 2200 50  0000 C CNN
+F 0 "D74" H 5900 2200 50  0000 C CNN
 F 1 "LED" H 6200 2200 50  0000 C CNN
 F 2 "LED_SMD:LED_0805_2012Metric" V 6000 2250 50  0001 C CNN
@@
 AR Path="/60E33DBC/5F767EF5/5F82FFCD/5F5C55CC" Ref="D87"  Part="1"
 AR Path="/60E33DBC/5F768DA1/5F82FFCD/5F5C55CC" Ref="D95"  Part="1"
-F 0 "D12" H 5700 2300 50  0000 C CNN
+F 0 "D71" H 5700 2300 50  0000 C CNN
 F 1 "LED" H 6000 2300 50  0000 C CNN
 F 2 "LED_SMD:LED_0805_2012Metric" V 5900 2350 50  0001 C CNN
@@
 AR Path="/60E33DBC/5F767EF5/5F82FFCD/5F5C55D2" Ref="D91"  Part="1"
 AR Path="/60E33DBC/5F768DA1/5F82FFCD/5F5C55D2" Ref="D99"  Part="1"
-F 0 "D16" H 5900 2400 50  0000 C CNN
+F 0 "D75" H 5900 2400 50  0000 C CNN
 F 1 "LED" H 6200 2400 50  0000 C CNN
 F 2 "LED_SMD:LED_0805_2012Metric" V 6000 2450 50  0001 C CNN
@@
 AR Path="/60E33DBC/5F767EF5/5F82FFCD/5F5C6722" Ref="D88"  Part="1"
 AR Path="/60E33DBC/5F768DA1/5F82FFCD/5F5C6722" Ref="D96"  Part="1"
-F 0 "D13" H 5700 2500 50  0000 C CNN
+F 0 "D72" H 5700 2500 50  0000 C CNN
 F 1 "LED" H 6000 2500 50  0000 C CNN
 F 2 "LED_SMD:LED_0805_2012Metric" V 5900 2550 50  0001 C CNN
@@
 AR Path="/60E33DBC/5F767EF5/5F82FFCD/5F5C6728" Ref="D92"  Part="1"
 AR Path="/60E33DBC/5F768DA1/5F82FFCD/5F5C6728" Ref="D100"  Part="1"
-F 0 "D17" H 5900 2600 50  0000 C CNN
+F 0 "D76" H 5900 2600 50  0000 C CNN
 F 1 "LED" H 6200 2600 50  0000 C CNN
 F 2 "LED_SMD:LED_0805_2012Metric" V 6000 2650 50  0001 C CNN
@@
 AR Path="/60E33DBC/5F767EF5/5F82FFCD/5F5C70EC" Ref="D89"  Part="1"
 AR Path="/60E33DBC/5F768DA1/5F82FFCD/5F5C70EC" Ref="D97"  Part="1"
-F 0 "D14" H 5700 2700 50  0000 C CNN
+F 0 "D73" H 5700 2700 50  0000 C CNN
 F 1 "LED" H 6000 2700 50  0000 C CNN
 F 2 "LED_SMD:LED_0805_2012Metric" V 5900 2750 50  0001 C CNN
@@
 AR Path="/60E33DBC/5F767EF5/5F82FFCD/5F5C70F2" Ref="D93"  Part="1"
 AR Path="/60E33DBC/5F768DA1/5F82FFCD/5F5C70F2" Ref="D101"  Part="1"
-F 0 "D18" H 5900 2800 50  0000 C CNN
+F 0 "D77" H 5900 2800 50  0000 C CNN
 F 1 "LED" H 6200 2800 50  0000 C CNN
 F 2 "LED_SMD:LED_0805_2012Metric" V 6000 2850 50  0001 C CNN
@@
 AR Path="/60E33DBC/5F767EF5/5F82FFCD/5F315EEA" Ref="U117"  Part="1"
 AR Path="/60E33DBC/5F768DA1/5F82FFCD/5F315EEA" Ref="U122"  Part="1"
-F 0 "U18" H 4600 3400 50  0000 C CNN
+F 0 "U107" H 4600 3400 50  0000 C CNN
 F 1 "74HC245" H 4700 3300 50  0000 C CNN
 F 2 "Package_SO:SSOP-20_5.3x7.2mm_P0.65mm" H 4500 2650 50  0001 C CNN
@@
 	1    0    0    -1
 $EndComp
+Text HLabel 3450 2000 0    50   Input ~ 0
+VAL[0..7]
 Wire Bus Line
 	3700 2000 3700 2750

Commit message: Schematic and Layout Done
Parts:
- removed C9: 0u1, Capacitor_SMD:C_0603_1608Metric, symbol Device:C_Small
- removed U8: 74HC245, Package_SO:SSOP-20_5.3x7.2mm_P0.65mm, symbol 74xx:74HC245
- D1, D2, D3, D4, D5, D6, D7, D8: footprint LED_SMD:LED_0805_2012Metric -> Diode_SMD:D_0603_1608Metric
Connections:
- net VAL0: now also R8.2
- net VAL1: now also R7.2
- net VAL2: now also R6.2
- net VAL3: now also R5.2
- net VAL4: now also R4.2
- net VAL5: now also R3.2
- net VAL6: now also R2.2
- net VAL7: now also R1.2
Other:
- moved on the sheet: D20, D21, D22, D23, D24, D25, D26, D27, R20, R21, R22, R23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
