File: KiCad/psMCU/ClockCtrlUI.sch (KiCad schematic (older format))
At the start: 22 parts

Commit message: Started work on schematic
Changed lines of the file:
@@
 $Descr A4 11693 8268
 encoding utf-8
-Sheet 19 65
+Sheet 16 94
 Title ""
 Date ""
@@
 S 5700 4100 700  200
 U 5F0227B2
-F0 "Do_Clock_Step" 50
+F0 "LED: Do_Clock_Step" 50
 F1 "1BitLED.sch" 50
 F2 "VAL" I L 5700 4200 50
@@
 S 3600 1950 700  200
 U 5F0227B5
-F0 "Clock_Step" 50
+F0 "LED: Clock_Step" 50
 F1 "1BitLED.sch" 50
 F2 "VAL" I L 3600 2050 50
@@
 S 3800 5150 700  200
 U 5F03D817
-F0 "Reset" 50
+F0 "LED: Reset" 50
 F1 "1BitLED.sch" 50
 F2 "VAL" I L 3800 5250 50
