File: KiCad/psMCU/BTN_TRIG.sch (KiCad schematic (older format))
At the start: 9 parts

Commit message: Added some footprints, small optimisations
Parts:
- U? (x2): footprint (none) -> Package_TO_SOT_SMD:SOT-353_SC-70-5
Changed lines of the file:
@@
 F 0 "U?" H 3050 1750 50  0000 C CNN
 F 1 "74LVC1G17" H 3200 1650 50  0000 C CNN
-F 2 "" H 2900 1800 50  0001 C CNN
+F 2 "Package_TO_SOT_SMD:SOT-353_SC-70-5" H 2900 1800 50  0001 C CNN
 F 3 "http://www.ti.com/lit/sg/scyt129e/scyt129e.pdf" H 2900 1800 50  0001 C CNN
 	1    2900 1800
@@
 F 0 "U?" H 4150 1750 50  0000 C CNN
 F 1 "74LVC1G32" H 4300 1650 50  0000 C CNN
-F 2 "" H 4000 1850 50  0001 C CNN
+F 2 "Package_TO_SOT_SMD:SOT-353_SC-70-5" H 4000 1850 50  0001 C CNN
 F 3 "http://www.ti.com/lit/sg/scyt129e/scyt129e.pdf" H 4000 1850 50  0001 C CNN
 	1    4000 1850

Commit message: Started some documentation work.
Other:
- note added: "BTN + Debounce"
- moved on the sheet: C?, R?, SW?, U?

Commit message: First Schematic Draft done.
Parts:
- C293, C294, C295: renamed from C?; footprint Capacitor_SMD:C_0603_1608Metric -> NoRef_Footprints:C_0603_1608Metric_NoRef
- R379, R380, R381: renamed from R?; footprint Resistor_SMD:R_0603_1608Metric -> NoRef_Footprints:D_0603_1608Metric_NoRef
- gave numbers to parts that had none: 3

Commit message: Small improvements.
Parts:
- renumbered C293 to C291, C294 to C292, C295 to C293, U286 to U284, U287 to U285
