File: KiCad/psMCU/Clock_Div.sch (KiCad schematic (older format))
At the start: 0 parts

Commit message: Pulled in from clock test, root layout first draft
Parts:
- added C33, C34, C35, C36, C37, C38, C39, C40, C41, C42, C43, C44, C55, C56: 0u1, Capacitor_SMD:C_0603_1608Metric, symbol Device:C_Small
- added U33: 74LVC1G04, Package_TO_SOT_SMD:SOT-353_SC-70-5, symbol 74xGxx:74LVC1G04
- added U34, U35, U36, U37, U38: 74HC161, Package_SO:SOIC-16_3.9x9.9mm_P1.27mm, symbol 74HC161:74HC161
- added U39, U40, U41, U42, U43: 74HC85, Package_SO:SOIC-16_3.9x9.9mm_P1.27mm, symbol 74xx:74LS85
- added U44: 74LVC1G32, Package_TO_SOT_SMD:SOT-353_SC-70-5, symbol 74xGxx:74LVC1G32
- added U55: 74LVC1G175, Package_TO_SOT_SMD:SOT-363_SC-70-6, symbol 74xGxx:74LVC1G175
- added U56: 74LVC1G86, Package_TO_SOT_SMD:SOT-353_SC-70-5, symbol 74xGxx:74LVC1G86
Connections:
- net CONT_CLK: now also U55.4 (Q), U56.2
- net OSC_IN: now also U34.2 (CLK), U35.2 (CLK), U36.2 (CLK), U37.2 (CLK), U38.2 (CLK), U55.1 (C)
- new net: U33.4, U34.10 (ENT), U34.7 (ENP), U34.9 (LOAD), U35.7 (ENP), U35.9 (LOAD), U36.7 (ENP), U36.9 (LOAD), U37.7 (ENP), U37.9 (LOAD), U38.7 (ENP), U38.9 (LOAD)
- new net: U34.15 (TC), U35.10 (ENT)
- new net: U35.15 (TC), U36.10 (ENT)
- new net: U36.15 (TC), U37.10 (ENT)
- new net: U37.15 (TC), U38.10 (ENT)
- new net: U33.2, U44.4, U56.1
- new net: U55.3 (D), U56.4
- new net: U39.7 (Oa<b), U40.2 (Ia<b)
- new net: U39.6 (Oa=b), U40.3 (Ia=b)
- new net: U39.5 (Oa>b), U40.4 (Ia>b)
- new net: U40.5 (Oa>b), U41.4 (Ia>b)
- new net: U40.6 (Oa=b), U41.3 (Ia=b)
- new net: U40.7 (Oa<b), U41.2 (Ia<b)
- new net: U41.5 (Oa>b), U42.4 (Ia>b)
- new net: U41.6 (Oa=b), U42.3 (Ia=b)
- new net: U41.7 (Oa<b), U42.2 (Ia<b)
- new net: U42.5 (Oa>b), U43.4 (Ia>b)
- new net: U42.6 (Oa=b), U43.3 (Ia=b)
- new net: U42.7 (Oa<b), U43.2 (Ia<b)
- new net: U43.6 (Oa=b), U44.2
- new net: U43.7 (Oa<b), U44.1
- new net +5V: C33.2, C34.2, C35.2, C36.2, C37.2, C38.2, C39.2, C40.2, C41.2, C42.2, C43.2, C44.2, C55.2, C56.2, U33.5 (VCC), U34.1 (CLR), U34.16 (VCC), U35.1 (CLR), U35.16 (VCC), U36.1 (CLR), U36.16 (VCC), U37.1 (CLR), U37.16 (VCC), U38.1 (CLR), U38.16 (VCC), U39.16 (VCC), U39.3 (Ia=b), U40.16 (VCC), U41.16 (VCC), U42.16 (VCC), U43.16 (VCC), U44.5 (VCC), U55.5 (VCC), U55.6 (~CLR), U56.5 (VCC)
- new net C0: U34.14 (Q0), U39.9 (B0)
- new net C1: U34.13 (Q1), U39.11 (B1)
- new net C10: U36.12 (Q2), U41.14 (B2)
- new net C11: U36.11 (Q3), U41.1 (B3)
- new net C12: U37.14 (Q0), U42.9 (B0)
- new net C13: U37.13 (Q1), U42.11 (B1)
- new net C14: U37.12 (Q2), U42.14 (B2)
- new net C15: U37.11 (Q3), U42.1 (B3)
- new net C16: U38.14 (Q0), U43.9 (B0)
- new net C17: U38.13 (Q1), U43.11 (B1)
- new net C18: U38.12 (Q2), U43.14 (B2)
- new net C19: U38.11 (Q3), U43.1 (B3)
- new net C2: U34.12 (Q2), U39.14 (B2)
- new net C3: U34.11 (Q3), U39.1 (B3)
- new net C4: U35.14 (Q0), U40.9 (B0)
- new net C5: U35.13 (Q1), U40.11 (B1)
- new net C6: U35.12 (Q2), U40.14 (B2)
- new net C7: U35.11 (Q3), U40.1 (B3)
- new net C8: U36.14 (Q0), U41.9 (B0)
- new net C9: U36.13 (Q1), U41.11 (B1)
- new net COMP0: U39.10 (A0)
- new net COMP1: U39.12 (A1)
- new net COMP13: U42.12 (A1)
- new net COMP17: U43.12 (A1)
- new net COMP19: U43.15 (A3)
- new net COMP5: U40.12 (A1)
- new net COMP9: U41.12 (A1)
- new net GND: C33.1, C34.1, C35.1, C36.1, C37.1, C38.1, C39.1, C40.1, C41.1, C42.1, C43.1, C44.1, C55.1, C56.1, U33.3 (GND), U34.3 (D0), U34.4 (D1), U34.5 (D2), U34.6 (D3), U34.8 (GND), U35.3 (D0), U35.4 (D1), U35.5 (D2), U35.6 (D3), U35.8 (GND), U36.3 (D0), U36.4 (D1), U36.5 (D2), U36.6 (D3), U36.8 (GND), U37.3 (D0), U37.4 (D1), U37.5 (D2), U37.6 (D3), U37.8 (GND), U38.3 (D0), U38.4 (D1), U38.5 (D2), U38.6 (D3), U38.8 (GND), U39.13 (A2), U39.15 (A3), U39.2 (Ia<b), U39.4 (Ia>b), U39.8 (GND), U40.10 (A0), U40.13 (A2), U40.15 (A3), U40.8 (GND), U41.10 (A0), U41.13 (A2), U41.15 (A3), U41.8 (GND), U42.10 (A0), U42.13 (A2), U42.15 (A3), U42.8 (GND), U43.10 (A0), U43.13 (A2), U43.8 (GND), U44.3 (GND), U55.2 (GND), U56.3 (GND)
- no-connect marks 0 -> 2
Other:
- note added: "T-FF with enable."

Commit message: Removed accidental anotation
Parts:
- renumbered C34 to C?, C35 to C?, C36 to C?, C37 to C?, C33 to C?, C56 to C?, C55 to C?, C38 to C?, C39 to C?, C40 to C?, C41 to C?, C42 to C?, C43 to C?, C44 to C?, U34 to U?, U35 to U?, U36 to U?, U37 to U?, U33 to U?, U55 to U?, U56 to U?, U38 to U?, U40 to U?, U39 to U?, U41 to U?, U42 to U?, U43 to U?, U44 to U?

Commit message: Started some documentation work.
Other:
- note added: "Comparator"
- note added: "Convert Frequency Setting\nto Comparator setpoint"
- note added: "Counter"
- note added: "Fastest setting, comparing to 0x0."
- note added: "Output T-FF"
- note removed: "T-FF with enable."
- moved on the sheet: C?, U?

Commit message: First Schematic Draft done.
Parts:
- C350, C351, C352, C353, C354, C355, C356, C357, C358, C359, C360, C361, C362, C363: renamed from C?; footprint Capacitor_SMD:C_0603_1608Metric -> NoRef_Footprints:C_0603_1608Metric_NoRef
- gave numbers to parts that had none: 14

Commit message: Small improvements.
Parts:
- renumbered C350 to C348, C351 to C349, C352 to C350, C353 to C351, C354 to C352, C355 to C353, C356 to C354, C357 to C355, C358 to C356, C359 to C357, C360 to C358, C361 to C359, C362 to C360, C363 to C361, U334 to U332, U335 to U333, U336 to U334, U337 to U335, U338 to U336, U339 to U337, U340 to U338, U341 to U339, U342 to U340, U343 to U341, U344 to U342, U345 to U343, U346 to U344, U347 to U345
