File: KiCad/psMCU/psMCU.kicad_pcb (KiCad board)
At the start: 2 copper layers, 0 parts

Commit message: Cleanup, ready for specific component values.
Parts:
- added REF**: SSOP-20_5.3x7.2mm_P0.65mm, Package_SO:SSOP-20_5.3x7.2mm_P0.65mm, F.Cu at (98.2, 90.7)
- added REF**: TSSOP-20_4.4x6.5mm_P0.65mm, Package_SO:TSSOP-20_4.4x6.5mm_P0.65mm, F.Cu at (98.4, 69.2)
Other:
- board text added: "DB"
- board text added: "PWR"
- board text added: "SSOP"
- board text added: "SSOP-20_5.3x7.2mm_P0.65mm"
- board text added: "TSSOP"
- board text added: "TSSOP-20_4.4x6.5mm_P0.65mm"
Changed lines of the file:
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@@
-(kicad_pcb (version 20171130) (host pcbnew "(5.1.5)-3")
+(kicad_pcb (version 20171130) (host pcbnew "(5.1.9)-1")
   (general
     (thickness 1.6)
-    (drawings 0)
+    (drawings 6)
     (tracks 0)
     (zones 0)
-    (modules 0)
+    (modules 2)
     (nets 1)
   )
@@
     (uvia_drill 0.1)
   )
+  (module Package_SO:SSOP-20_5.3x7.2mm_P0.65mm (layer F.Cu)
+    (at 98.171 90.7034)
+    (descr "SSOP, 20 Pin (http://ww1.microchip.com/downloads/en/DeviceDoc/40001800C.pdf), generated with kicad-footprint-generator ipc_gullwing_generator.py")
+    (tags "SSOP SO")
+    (attr smd)
+    (fp_text reference REF** (at 0 -4.55) (layer F.SilkS)
+      (effects (font (size 1 1) (thickness 0.15)))
+    )
+    (fp_text value SSOP-20_5.3x7.2mm_P0.65mm (at 0 4.55) (layer F.Fab)
+      (effects (font (size 1 1) (thickness 0.15)))
+    )
+    (fp_text user %R (at 0 0) (layer F.Fab)
+      (effects (font (size 1 1) (thickness 0.15)))
+    )
+    (fp_line (start 0 3.71) (end 2.76 3.71) (layer F.SilkS) (width 0.12))
+    (fp_line (start 2.76 3.71) (end 2.76 3.435) (layer F.SilkS) (width 0.12))
+    (fp_line (start 0 3.71) (end -2.76 3.71) (layer F.SilkS) (width 0.12))
+    (fp_line (start -2.76 3.71) (end -2.76 3.435) (layer F.SilkS) (width 0.12))
+    (fp_line (start 0 -3.71) (end 2.76 -3.71) (layer F.SilkS) (width 0.12))
+    (fp_line (start 2.76 -3.71) (end 2.76 -3.435) (layer F.SilkS) (width 0.12))
+    (fp_line (start 0 -3.71) (end -2.76 -3.71) (layer F.SilkS) (width 0.12))
+    (fp_line (start -2.76 -3.71) (end -2.76 -3.435) (layer F.SilkS) (width 0.12))
+    (fp_line (start -2.76 -3.435) (end -4.45 -3.435) (layer F.SilkS) (width 0.12))
+    (fp_line (start -1.65 -3.6) (end 2.65 -3.6) (layer F.Fab) (width 0.1))
+    (fp_line (start 2.65 -3.6) (end 2.65 3.6) (layer F.Fab) (width 0.1))
+    (fp_line (start 2.65 3.6) (end -2.65 3.6) (layer F.Fab) (width 0.1))
+    (fp_line (start -2.65 3.6) (end -2.65 -2.6) (layer F.Fab) (width 0.1))
+    (fp_line (start -2.65 -2.6) (end -1.65 -3.6) (layer F.Fab) (width 0.1))
+    (fp_line (start -4.7 -3.85) (end -4.7 3.85) (layer F.CrtYd) (width 0.05))
+    (fp_line (start -4.7 3.85) (end 4.7 3.85) (layer F.CrtYd) (width 0.05))
+    (fp_line (start 4.7 3.85) (end 4.7 -3.85) (layer F.CrtYd) (width 0.05))
+    (fp_line (start 4.7 -3.85) (end -4.7 -3.85) (layer F.CrtYd) (width 0.05))
+    (pad 20 smd roundrect (at 3.5 -2.925) (size 1.9 0.5) (layers F.Cu F.Paste F.Mask) (roundrect_rratio 0.25))
+    (pad 19 smd roundrect (at 3.5 -2.275) (size 1.9 0.5) (layers F.Cu F.Paste F.Mask) (roundrect_rratio 0.25))
+    (pad 18 smd roundrect (at 3.5 -1.625) (size 1.9 0.5) (layers F.Cu F.Paste F.Mask) (roundrect_rratio 0.25))
+    (pad 17 smd roundrect (at 3.5 -0.975) (size 1.9 0.5) (layers F.Cu F.Paste F.Mask) (roundrect_rratio 0.25))
+    (pad 16 smd roundrect (at 3.5 -0.325) (size 1.9 0.5) (layers F.Cu F.Paste F.Mask) (roundrect_rratio 0.25))
+    (pad 15 smd roundrect (at 3.5 0.325) (size 1.9 0.5) (layers F.Cu F.Paste F.Mask) (roundrect_rratio 0.25))
+    (pad 14 smd roundrect (at 3.5 0.975) (size 1.9 0.5) (layers F.Cu F.Paste F.Mask) (roundrect_rratio 0.25))
+    (pad 13 smd roundrect (at 3.5 1.625) (size 1.9 0.5) (layers F.Cu F.Paste F.Mask) (roundrect_rratio 0.25))
+    (pad 12 smd roundrect (at 3.5 2.275) (size 1.9 0.5) (layers F.Cu F.Paste F.Mask) (roundrect_rratio 0.25))
+    (pad 11 smd roundrect (at 3.5 2.925) (size 1.9 0.5) (layers F.Cu F.Paste F.Mask) (roundrect_rratio 0.25))
+    (pad 10 smd roundrect (at -3.5 2.925) (size 1.9 0.5) (layers F.Cu F.Paste F.Mask) (roundrect_rratio 0.25))
+    (pad 9 smd roundrect (at -3.5 2.275) (size 1.9 0.5) (layers F.Cu F.Paste F.Mask) (roundrect_rratio 0.25))
+    (pad 8 smd roundrect (at -3.5 1.625) (size 1.9 0.5) (layers F.Cu F.Paste F.Mask) (roundrect_rratio 0.25))
+    (pad 7 smd roundrect (at -3.5 0.975) (size 1.9 0.5) (layers F.Cu F.Paste F.Mask) (roundrect_rratio 0.25))
+    (pad 6 smd roundrect (at -3.5 0.325) (size 1.9 0.5) (layers F.Cu F.Paste F.Mask) (roundrect_rratio 0.25))
+    (pad 5 smd roundrect (at -3.5 -0.325) (size 1.9 0.5) (layers F.Cu F.Paste F.Mask) (roundrect_rratio 0.25))
+    (pad 4 smd roundrect (at -3.5 -0.975) (size 1.9 0.5) (layers F.Cu F.Paste F.Mask) (roundrect_rratio 0.25))
+    (pad 3 smd roundrect (at -3.5 -1.625) (size 1.9 0.5) (layers F.Cu F.Paste F.Mask) (roundrect_rratio 0.25))
+    (pad 2 smd roundrect (at -3.5 -2.275) (size 1.9 0.5) (layers F.Cu F.Paste F.Mask) (roundrect_rratio 0.25))
+    (pad 1 smd roundrect (at -3.5 -2.925) (size 1.9 0.5) (layers F.Cu F.Paste F.Mask) (roundrect_rratio 0.25))
+    (model ${KISYS3DMOD}/Package_SO.3dshapes/SSOP-20_5.3x7.2mm_P0.65mm.wrl
+      (at (xyz 0 0 0))
+      (scale (xyz 1 1 1))
+      (rotate (xyz 0 0 0))
+    )
+  )
+  (module Package_SO:TSSOP-20_4.4x6.5mm_P0.65mm (layer F.Cu)
+    (at 98.425 69.215)
+    (descr "TSSOP, 20 Pin (JEDEC MO-153 Var AC https://www.jedec.org/document_search?search_api_views_fulltext=MO-153), generated with kicad-footprint-generator ipc_gullwing_generator.py")
+    (tags "TSSOP SO")
+    (attr smd)
+    (fp_text reference REF** (at 0 -4.2) (layer F.SilkS)
+      (effects (font (size 1 1) (thickness 0.15)))
+    )
+    (fp_text value TSSOP-20_4.4x6.5mm_P0.65mm (at 0 4.2) (layer F.Fab)
+      (effects (font (size 1 1) (thickness 0.15)))
+    )
+    (fp_text user %R (at 0 0) (layer F.Fab)
+      (effects (font (size 1 1) (thickness 0.15)))
+    )
+    (fp_line (start 0 3.385) (end 2.2 3.385) (layer F.SilkS) (width 0.12))
+    (fp_line (start 0 3.385) (end -2.2 3.385) (layer F.SilkS) (width 0.12))
+    (fp_line (start 0 -3.385) (end 2.2 -3.385) (layer F.SilkS) (width 0.12))
+    (fp_line (start 0 -3.385) (end -3.6 -3.385) (layer F.SilkS) (width 0.12))
+    (fp_line (start -1.2 -3.25) (end 2.2 -3.25) (layer F.Fab) (width 0.1))
+    (fp_line (start 2.2 -3.25) (end 2.2 3.25) (layer F.Fab) (width 0.1))
+    (fp_line (start 2.2 3.25) (end -2.2 3.25) (layer F.Fab) (width 0.1))
+    (fp_line (start -2.2 3.25) (end -2.2 -2.25) (layer F.Fab) (width 0.1))
+    (fp_line (start -2.2 -2.25) (end -1.2 -3.25) (layer F.Fab) (width 0.1))
+    (fp_line (start -3.85 -3.5) (end -3.85 3.5) (layer F.CrtYd) (width 0.05))
+    (fp_line (start -3.85 3.5) (end 3.85 3.5) (layer F.CrtYd) (width 0.05))
+    (fp_line (start 3.85 3.5) (end 3.85 -3.5) (layer F.CrtYd) (width 0.05))
+    (fp_line (start 3.85 -3.5) (end -3.85 -3.5) (layer F.CrtYd) (width 0.05))
+    (pad 20 smd roundrect (at 2.8625 -2.925) (size 1.475 0.4) (layers F.Cu F.Paste F.Mask) (roundrect_rratio 0.25))
+    (pad 19 smd roundrect (at 2.8625 -2.275) (size 1.475 0.4) (layers F.Cu F.Paste F.Mask) (roundrect_rratio 0.25))
+    (pad 18 smd roundrect (at 2.8625 -1.625) (size 1.475 0.4) (layers F.Cu F.Paste F.Mask) (roundrect_rratio 0.25))
+    (pad 17 smd roundrect (at 2.8625 -0.975) (size 1.475 0.4) (layers F.Cu F.Paste F.Mask) (roundrect_rratio 0.25))
+    (pad 16 smd roundrect (at 2.8625 -0.325) (size 1.475 0.4) (layers F.Cu F.Paste F.Mask) (roundrect_rratio 0.25))
+    (pad 15 smd roundrect (at 2.8625 0.325) (size 1.475 0.4) (layers F.Cu F.Paste F.Mask) (roundrect_rratio 0.25))
+    (pad 14 smd roundrect (at 2.8625 0.975) (size 1.475 0.4) (layers F.Cu F.Paste F.Mask) (roundrect_rratio 0.25))
+    (pad 13 smd roundrect (at 2.8625 1.625) (size 1.475 0.4) (layers F.Cu F.Paste F.Mask) (roundrect_rratio 0.25))
+    (pad 12 smd roundrect (at 2.8625 2.275) (size 1.475 0.4) (layers F.Cu F.Paste F.Mask) (roundrect_rratio 0.25))
+    (pad 11 smd roundrect (at 2.8625 2.925) (size 1.475 0.4) (layers F.Cu F.Paste F.Mask) (roundrect_rratio 0.25))
+    (pad 10 smd roundrect (at -2.8625 2.925) (size 1.475 0.4) (layers F.Cu F.Paste F.Mask) (roundrect_rratio 0.25))
+    (pad 9 smd roundrect (at -2.8625 2.275) (size 1.475 0.4) (layers F.Cu F.Paste F.Mask) (roundrect_rratio 0.25))
+    (pad 8 smd roundrect (at -2.8625 1.625) (size 1.475 0.4) (layers F.Cu F.Paste F.Mask) (roundrect_rratio 0.25))
+    (pad 7 smd roundrect (at -2.8625 0.975) (size 1.475 0.4) (layers F.Cu F.Paste F.Mask) (roundrect_rratio 0.25))
+    (pad 6 smd roundrect (at -2.8625 0.325) (size 1.475 0.4) (layers F.Cu F.Paste F.Mask) (roundrect_rratio 0.25))
+    (pad 5 smd roundrect (at -2.8625 -0.325) (size 1.475 0.4) (layers F.Cu F.Paste F.Mask) (roundrect_rratio 0.25))
+    (pad 4 smd roundrect (at -2.8625 -0.975) (size 1.475 0.4) (layers F.Cu F.Paste F.Mask) (roundrect_rratio 0.25))
+    (pad 3 smd roundrect (at -2.8625 -1.625) (size 1.475 0.4) (layers F.Cu F.Paste F.Mask) (roundrect_rratio 0.25))
+    (pad 2 smd roundrect (at -2.8625 -2.275) (size 1.475 0.4) (layers F.Cu F.Paste F.Mask) (roundrect_rratio 0.25))
+    (pad 1 smd roundrect (at -2.8625 -2.925) (size 1.475 0.4) (layers F.Cu F.Paste F.Mask) (roundrect_rratio 0.25))
+    (model ${KISYS3DMOD}/Package_SO.3dshapes/TSSOP-20_4.4x6.5mm_P0.65mm.wrl
+      (at (xyz 0 0 0))
+      (scale (xyz 1 1 1))
+      (rotate (xyz 0 0 0))
+    )
+  )
+  (gr_text SSOP-20_5.3x7.2mm_P0.65mm (at 98.4758 98.2218) (layer F.Cu)
+    (effects (font (size 1.5 1.5) (thickness 0.3)))
+  )
+  (gr_text TSSOP-20_4.4x6.5mm_P0.65mm (at 98.5266 76.8096) (layer F.Cu)
+    (effects (font (size 1.5 1.5) (thickness 0.3)))
+  )
+  (gr_text DB (at 98.3996 96.0374) (layer F.Cu)
+    (effects (font (size 1.5 1.5) (thickness 0.3)))
+  )
+  (gr_text PWR (at 98.4504 74.5744) (layer F.Cu)
+    (effects (font (size 1.5 1.5) (thickness 0.3)))
+  )
+  (gr_text TSSOP (at 98.425 62.865) (layer F.Cu)
+    (effects (font (size 1.5 1.5) (thickness 0.3)))
+  )
+  (gr_text SSOP (at 98.3488 84.0232) (layer F.Cu)
+    (effects (font (size 1.5 1.5) (thickness 0.3)))
+  )
 )

Commit message: ERC clean.
Parts:
- removed REF**: SSOP-20_5.3x7.2mm_P0.65mm, Package_SO:SSOP-20_5.3x7.2mm_P0.65mm
- removed REF**: TSSOP-20_4.4x6.5mm_P0.65mm, Package_SO:TSSOP-20_4.4x6.5mm_P0.65mm
Other:
- board text removed: "DB"
- board text removed: "PWR"
- board text removed: "SSOP"
- board text removed: "SSOP-20_5.3x7.2mm_P0.65mm"
- board text removed: "TSSOP"
- board text removed: "TSSOP-20_4.4x6.5mm_P0.65mm"
Changed lines of the file:
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@@
   (general
     (thickness 1.6)
-    (drawings 6)
+    (drawings 0)
     (tracks 0)
     (zones 0)
-    (modules 2)
+    (modules 0)
     (nets 1)
   )
@@
     (uvia_drill 0.1)
   )
-  (module Package_SO:SSOP-20_5.3x7.2mm_P0.65mm (layer F.Cu)
-    (at 98.171 90.7034)
-    (descr "SSOP, 20 Pin (http://ww1.microchip.com/downloads/en/DeviceDoc/40001800C.pdf), generated with kicad-footprint-generator ipc_gullwing_generator.py")
-    (tags "SSOP SO")
-    (attr smd)
-    (fp_text reference REF** (at 0 -4.55) (layer F.SilkS)
-      (effects (font (size 1 1) (thickness 0.15)))
-    )
-    (fp_text value SSOP-20_5.3x7.2mm_P0.65mm (at 0 4.55) (layer F.Fab)
-      (effects (font (size 1 1) (thickness 0.15)))
-    )
-    (fp_text user %R (at 0 0) (layer F.Fab)
-      (effects (font (size 1 1) (thickness 0.15)))
-    )
-    (fp_line (start 0 3.71) (end 2.76 3.71) (layer F.SilkS) (width 0.12))
-    (fp_line (start 2.76 3.71) (end 2.76 3.435) (layer F.SilkS) (width 0.12))
-    (fp_line (start 0 3.71) (end -2.76 3.71) (layer F.SilkS) (width 0.12))
-    (fp_line (start -2.76 3.71) (end -2.76 3.435) (layer F.SilkS) (width 0.12))
-    (fp_line (start 0 -3.71) (end 2.76 -3.71) (layer F.SilkS) (width 0.12))
-    (fp_line (start 2.76 -3.71) (end 2.76 -3.435) (layer F.SilkS) (width 0.12))
-    (fp_line (start 0 -3.71) (end -2.76 -3.71) (layer F.SilkS) (width 0.12))
-    (fp_line (start -2.76 -3.71) (end -2.76 -3.435) (layer F.SilkS) (width 0.12))
-    (fp_line (start -2.76 -3.435) (end -4.45 -3.435) (layer F.SilkS) (width 0.12))
-    (fp_line (start -1.65 -3.6) (end 2.65 -3.6) (layer F.Fab) (width 0.1))
-    (fp_line (start 2.65 -3.6) (end 2.65 3.6) (layer F.Fab) (width 0.1))
-    (fp_line (start 2.65 3.6) (end -2.65 3.6) (layer F.Fab) (width 0.1))
-    (fp_line (start -2.65 3.6) (end -2.65 -2.6) (layer F.Fab) (width 0.1))
-    (fp_line (start -2.65 -2.6) (end -1.65 -3.6) (layer F.Fab) (width 0.1))
-    (fp_line (start -4.7 -3.85) (end -4.7 3.85) (layer F.CrtYd) (width 0.05))
-    (fp_line (start -4.7 3.85) (end 4.7 3.85) (layer F.CrtYd) (width 0.05))
-    (fp_line (start 4.7 3.85) (end 4.7 -3.85) (layer F.CrtYd) (width 0.05))
-    (fp_line (start 4.7 -3.85) (end -4.7 -3.85) (layer F.CrtYd) (width 0.05))
-    (pad 20 smd roundrect (at 3.5 -2.925) (size 1.9 0.5) (layers F.Cu F.Paste F.Mask) (roundrect_rratio 0.25))
-    (pad 19 smd roundrect (at 3.5 -2.275) (size 1.9 0.5) (layers F.Cu F.Paste F.Mask) (roundrect_rratio 0.25))
-    (pad 18 smd roundrect (at 3.5 -1.625) (size 1.9 0.5) (layers F.Cu F.Paste F.Mask) (roundrect_rratio 0.25))
-    (pad 17 smd roundrect (at 3.5 -0.975) (size 1.9 0.5) (layers F.Cu F.Paste F.Mask) (roundrect_rratio 0.25))
-    (pad 16 smd roundrect (at 3.5 -0.325) (size 1.9 0.5) (layers F.Cu F.Paste F.Mask) (roundrect_rratio 0.25))
-    (pad 15 smd roundrect (at 3.5 0.325) (size 1.9 0.5) (layers F.Cu F.Paste F.Mask) (roundrect_rratio 0.25))
-    (pad 14 smd roundrect (at 3.5 0.975) (size 1.9 0.5) (layers F.Cu F.Paste F.Mask) (roundrect_rratio 0.25))
-    (pad 13 smd roundrect (at 3.5 1.625) (size 1.9 0.5) (layers F.Cu F.Paste F.Mask) (roundrect_rratio 0.25))
-    (pad 12 smd roundrect (at 3.5 2.275) (size 1.9 0.5) (layers F.Cu F.Paste F.Mask) (roundrect_rratio 0.25))
-    (pad 11 smd roundrect (at 3.5 2.925) (size 1.9 0.5) (layers F.Cu F.Paste F.Mask) (roundrect_rratio 0.25))
-    (pad 10 smd roundrect (at -3.5 2.925) (size 1.9 0.5) (layers F.Cu F.Paste F.Mask) (roundrect_rratio 0.25))
-    (pad 9 smd roundrect (at -3.5 2.275) (size 1.9 0.5) (layers F.Cu F.Paste F.Mask) (roundrect_rratio 0.25))
-    (pad 8 smd roundrect (at -3.5 1.625) (size 1.9 0.5) (layers F.Cu F.Paste F.Mask) (roundrect_rratio 0.25))
-    (pad 7 smd roundrect (at -3.5 0.975) (size 1.9 0.5) (layers F.Cu F.Paste F.Mask) (roundrect_rratio 0.25))
-    (pad 6 smd roundrect (at -3.5 0.325) (size 1.9 0.5) (layers F.Cu F.Paste F.Mask) (roundrect_rratio 0.25))
-    (pad 5 smd roundrect (at -3.5 -0.325) (size 1.9 0.5) (layers F.Cu F.Paste F.Mask) (roundrect_rratio 0.25))
-    (pad 4 smd roundrect (at -3.5 -0.975) (size 1.9 0.5) (layers F.Cu F.Paste F.Mask) (roundrect_rratio 0.25))
-    (pad 3 smd roundrect (at -3.5 -1.625) (size 1.9 0.5) (layers F.Cu F.Paste F.Mask) (roundrect_rratio 0.25))
-    (pad 2 smd roundrect (at -3.5 -2.275) (size 1.9 0.5) (layers F.Cu F.Paste F.Mask) (roundrect_rratio 0.25))
-    (pad 1 smd roundrect (at -3.5 -2.925) (size 1.9 0.5) (layers F.Cu F.Paste F.Mask) (roundrect_rratio 0.25))
-    (model ${KISYS3DMOD}/Package_SO.3dshapes/SSOP-20_5.3x7.2mm_P0.65mm.wrl
-      (at (xyz 0 0 0))
-      (scale (xyz 1 1 1))
-      (rotate (xyz 0 0 0))
-    )
-  )
-  (module Package_SO:TSSOP-20_4.4x6.5mm_P0.65mm (layer F.Cu)
-    (at 98.425 69.215)
-    (descr "TSSOP, 20 Pin (JEDEC MO-153 Var AC https://www.jedec.org/document_search?search_api_views_fulltext=MO-153), generated with kicad-footprint-generator ipc_gullwing_generator.py")
-    (tags "TSSOP SO")
-    (attr smd)
-    (fp_text reference REF** (at 0 -4.2) (layer F.SilkS)
-      (effects (font (size 1 1) (thickness 0.15)))
-    )
-    (fp_text value TSSOP-20_4.4x6.5mm_P0.65mm (at 0 4.2) (layer F.Fab)
-      (effects (font (size 1 1) (thickness 0.15)))
-    )
-    (fp_text user %R (at 0 0) (layer F.Fab)
-      (effects (font (size 1 1) (thickness 0.15)))
-    )
-    (fp_line (start 0 3.385) (end 2.2 3.385) (layer F.SilkS) (width 0.12))
-    (fp_line (start 0 3.385) (end -2.2 3.385) (layer F.SilkS) (width 0.12))
-    (fp_line (start 0 -3.385) (end 2.2 -3.385) (layer F.SilkS) (width 0.12))
-    (fp_line (start 0 -3.385) (end -3.6 -3.385) (layer F.SilkS) (width 0.12))
-    (fp_line (start -1.2 -3.25) (end 2.2 -3.25) (layer F.Fab) (width 0.1))
-    (fp_line (start 2.2 -3.25) (end 2.2 3.25) (layer F.Fab) (width 0.1))
-    (fp_line (start 2.2 3.25) (end -2.2 3.25) (layer F.Fab) (width 0.1))
-    (fp_line (start -2.2 3.25) (end -2.2 -2.25) (layer F.Fab) (width 0.1))
-    (fp_line (start -2.2 -2.25) (end -1.2 -3.25) (layer F.Fab) (width 0.1))
-    (fp_line (start -3.85 -3.5) (end -3.85 3.5) (layer F.CrtYd) (width 0.05))
-    (fp_line (start -3.85 3.5) (end 3.85 3.5) (layer F.CrtYd) (width 0.05))
-    (fp_line (start 3.85 3.5) (end 3.85 -3.5) (layer F.CrtYd) (width 0.05))
-    (fp_line (start 3.85 -3.5) (end -3.85 -3.5) (layer F.CrtYd) (width 0.05))
-    (pad 20 smd roundrect (at 2.8625 -2.925) (size 1.475 0.4) (layers F.Cu F.Paste F.Mask) (roundrect_rratio 0.25))
-    (pad 19 smd roundrect (at 2.8625 -2.275) (size 1.475 0.4) (layers F.Cu F.Paste F.Mask) (roundrect_rratio 0.25))
-    (pad 18 smd roundrect (at 2.8625 -1.625) (size 1.475 0.4) (layers F.Cu F.Paste F.Mask) (roundrect_rratio 0.25))
-    (pad 17 smd roundrect (at 2.8625 -0.975) (size 1.475 0.4) (layers F.Cu F.Paste F.Mask) (roundrect_rratio 0.25))
-    (pad 16 smd roundrect (at 2.8625 -0.325) (size 1.475 0.4) (layers F.Cu F.Paste F.Mask) (roundrect_rratio 0.25))
-    (pad 15 smd roundrect (at 2.8625 0.325) (size 1.475 0.4) (layers F.Cu F.Paste F.Mask) (roundrect_rratio 0.25))
-    (pad 14 smd roundrect (at 2.8625 0.975) (size 1.475 0.4) (layers F.Cu F.Paste F.Mask) (roundrect_rratio 0.25))
-    (pad 13 smd roundrect (at 2.8625 1.625) (size 1.475 0.4) (layers F.Cu F.Paste F.Mask) (roundrect_rratio 0.25))
-    (pad 12 smd roundrect (at 2.8625 2.275) (size 1.475 0.4) (layers F.Cu F.Paste F.Mask) (roundrect_rratio 0.25))
-    (pad 11 smd roundrect (at 2.8625 2.925) (size 1.475 0.4) (layers F.Cu F.Paste F.Mask) (roundrect_rratio 0.25))
-    (pad 10 smd roundrect (at -2.8625 2.925) (size 1.475 0.4) (layers F.Cu F.Paste F.Mask) (roundrect_rratio 0.25))
-    (pad 9 smd roundrect (at -2.8625 2.275) (size 1.475 0.4) (layers F.Cu F.Paste F.Mask) (roundrect_rratio 0.25))
-    (pad 8 smd roundrect (at -2.8625 1.625) (size 1.475 0.4) (layers F.Cu F.Paste F.Mask) (roundrect_rratio 0.25))
-    (pad 7 smd roundrect (at -2.8625 0.975) (size 1.475 0.4) (layers F.Cu F.Paste F.Mask) (roundrect_rratio 0.25))
-    (pad 6 smd roundrect (at -2.8625 0.325) (size 1.475 0.4) (layers F.Cu F.Paste F.Mask) (roundrect_rratio 0.25))
-    (pad 5 smd roundrect (at -2.8625 -0.325) (size 1.475 0.4) (layers F.Cu F.Paste F.Mask) (roundrect_rratio 0.25))
-    (pad 4 smd roundrect (at -2.8625 -0.975) (size 1.475 0.4) (layers F.Cu F.Paste F.Mask) (roundrect_rratio 0.25))
-    (pad 3 smd roundrect (at -2.8625 -1.625) (size 1.475 0.4) (layers F.Cu F.Paste F.Mask) (roundrect_rratio 0.25))
-    (pad 2 smd roundrect (at -2.8625 -2.275) (size 1.475 0.4) (layers F.Cu F.Paste F.Mask) (roundrect_rratio 0.25))
-    (pad 1 smd roundrect (at -2.8625 -2.925) (size 1.475 0.4) (layers F.Cu F.Paste F.Mask) (roundrect_rratio 0.25))
-    (model ${KISYS3DMOD}/Package_SO.3dshapes/TSSOP-20_4.4x6.5mm_P0.65mm.wrl
-      (at (xyz 0 0 0))
-      (scale (xyz 1 1 1))
-      (rotate (xyz 0 0 0))
-    )
-  )
-  (gr_text SSOP-20_5.3x7.2mm_P0.65mm (at 98.4758 98.2218) (layer F.Cu)
-    (effects (font (size 1.5 1.5) (thickness 0.3)))
-  )
-  (gr_text TSSOP-20_4.4x6.5mm_P0.65mm (at 98.5266 76.8096) (layer F.Cu)
-    (effects (font (size 1.5 1.5) (thickness 0.3)))
-  )
-  (gr_text DB (at 98.3996 96.0374) (layer F.Cu)
-    (effects (font (size 1.5 1.5) (thickness 0.3)))
-  )
-  (gr_text PWR (at 98.4504 74.5744) (layer F.Cu)
-    (effects (font (size 1.5 1.5) (thickness 0.3)))
-  )
-  (gr_text TSSOP (at 98.425 62.865) (layer F.Cu)
-    (effects (font (size 1.5 1.5) (thickness 0.3)))
-  )
-  (gr_text SSOP (at 98.3488 84.0232) (layer F.Cu)
-    (effects (font (size 1.5 1.5) (thickness 0.3)))
-  )
 )
