File: ECAD/psMCU/KiCad/Stack_ALU.sch (KiCad schematic (older format))
At the start: 8 parts

Commit message: Annotation.
Parts:
- gave numbers to parts that had none: 8
Changed lines of the file:
@@
 AR Path="/5F396002/627E93BB" Ref="U?"  Part="1"
 AR Path="/5FD6F26B/627E93BB" Ref="U?"  Part="1"
-AR Path="/5FD6EE9C/6118ACE0/627E93BB" Ref="U?"  Part="1"
-F 0 "U?" H 4400 2550 50  0000 C CNN
+AR Path="/5FD6EE9C/6118ACE0/627E93BB" Ref="U408"  Part="1"
+F 0 "U408" H 4400 2550 50  0000 C CNN
 F 1 "CD74HC283M96" H 4650 2450 50  0000 C CNN
 F 2 "Package_SO:SOIC-16_3.9x9.9mm_P1.27mm" H 4300 1800 50  0001 C CNN
@@
 AR Path="/5F396002/627E93C1" Ref="#PWR?"  Part="1"
 AR Path="/5FD6F26B/627E93C1" Ref="#PWR?"  Part="1"
-AR Path="/5FD6EE9C/6118ACE0/627E93C1" Ref="#PWR?"  Part="1"
-F 0 "#PWR?" H 4300 700 50  0001 C CNN
+AR Path="/5FD6EE9C/6118ACE0/627E93C1" Ref="#PWR01185"  Part="1"
+F 0 "#PWR01185" H 4300 700 50  0001 C CNN
 F 1 "+5V" H 4150 900 50  0000 C CNN
 F 2 "" H 4300 850 50  0001 C CNN
@@
 AR Path="/5F396002/627E93C9" Ref="#PWR?"  Part="1"
 AR Path="/5FD6F26B/627E93C9" Ref="#PWR?"  Part="1"
-AR Path="/5FD6EE9C/6118ACE0/627E93C9" Ref="#PWR?"  Part="1"
-F 0 "#PWR?" H 4600 650 50  0001 C CNN
+AR Path="/5FD6EE9C/6118ACE0/627E93C9" Ref="#PWR01193"  Part="1"
+F 0 "#PWR01193" H 4600 650 50  0001 C CNN
 F 1 "GND" V 4605 772 50  0000 R CNN
 F 2 "" H 4600 900 50  0001 C CNN
@@
 AR Path="/5F396002/627E93CF" Ref="C?"  Part="1"
 AR Path="/5FD6F26B/627E93CF" Ref="C?"  Part="1"
-AR Path="/5FD6EE9C/6118ACE0/627E93CF" Ref="C?"  Part="1"
-F 0 "C?" V 4221 900 50  0000 C CNN
+AR Path="/5FD6EE9C/6118ACE0/627E93CF" Ref="C421"  Part="1"
+F 0 "C421" V 4221 900 50  0000 C CNN
 F 1 "0u1" V 4312 900 50  0000 C CNN
 F 2 "NoRef_Footprints:C_0603_1608Metric_NoRef" H 4450 900 50  0001 C CNN
@@
 AR Path="/5F396002/627E93D8" Ref="#PWR?"  Part="1"
 AR Path="/5FD6F26B/627E93D8" Ref="#PWR?"  Part="1"
-AR Path="/5FD6EE9C/6118ACE0/627E93D8" Ref="#PWR?"  Part="1"
-F 0 "#PWR?" H 4300 2400 50  0001 C CNN
+AR Path="/5FD6EE9C/6118ACE0/627E93D8" Ref="#PWR01186"  Part="1"
+F 0 "#PWR01186" H 4300 2400 50  0001 C CNN
 F 1 "GND" H 4150 2600 50  0000 C CNN
 F 2 "" H 4300 2650 50  0001 C CNN
@@
 AR Path="/5F396002/627F4FD8" Ref="U?"  Part="1"
 AR Path="/5FD6F26B/627F4FD8" Ref="U?"  Part="1"
-AR Path="/5FD6EE9C/6118ACE0/627F4FD8" Ref="U?"  Part="1"
-F 0 "U?" H 4400 4800 50  0000 C CNN
+AR Path="/5FD6EE9C/6118ACE0/627F4FD8" Ref="U410"  Part="1"
+F 0 "U410" H 4400 4800 50  0000 C CNN
 F 1 "CD74HC283M96" H 4650 4700 50  0000 C CNN
 F 2 "Package_SO:SOIC-16_3.9x9.9mm_P1.27mm" H 4300 4050 50  0001 C CNN
@@
 AR Path="/5F396002/627F4FDE" Ref="#PWR?"  Part="1"
 AR Path="/5FD6F26B/627F4FDE" Ref="#PWR?"  Part="1"
-AR Path="/5FD6EE9C/6118ACE0/627F4FDE" Ref="#PWR?"  Part="1"
-F 0 "#PWR?" H 4300 2950 50  0001 C CNN
+AR Path="/5FD6EE9C/6118ACE0/627F4FDE" Ref="#PWR01187"  Part="1"
+F 0 "#PWR01187" H 4300 2950 50  0001 C CNN
 F 1 "+5V" H 4150 3150 50  0000 C CNN
 F 2 "" H 4300 3100 50  0001 C CNN
@@
 AR Path="/5F396002/627F4FE6" Ref="#PWR?"  Part="1"
 AR Path="/5FD6F26B/627F4FE6" Ref="#PWR?"  Part="1"
-AR Path="/5FD6EE9C/6118ACE0/627F4FE6" Ref="#PWR?"  Part="1"
-F 0 "#PWR?" H 4600 2900 50  0001 C CNN
+AR Path="/5FD6EE9C/6118ACE0/627F4FE6" Ref="#PWR01194"  Part="1"
+F 0 "#PWR01194" H 4600 2900 50  0001 C CNN
 F 1 "GND" V 4605 3022 50  0000 R CNN
 F 2 "" H 4600 3150 50  0001 C CNN
@@
 AR Path="/5F396002/627F4FEC" Ref="C?"  Part="1"
 AR Path="/5FD6F26B/627F4FEC" Ref="C?"  Part="1"
-AR Path="/5FD6EE9C/6118ACE0/627F4FEC" Ref="C?"  Part="1"
-F 0 "C?" V 4221 3150 50  0000 C CNN
+AR Path="/5FD6EE9C/6118ACE0/627F4FEC" Ref="C422"  Part="1"
+F 0 "C422" V 4221 3150 50  0000 C CNN
 F 1 "0u1" V 4312 3150 50  0000 C CNN
 F 2 "NoRef_Footprints:C_0603_1608Metric_NoRef" H 4450 3150 50  0001 C CNN
@@
 AR Path="/5F396002/627F4FF5" Ref="#PWR?"  Part="1"
 AR Path="/5FD6F26B/627F4FF5" Ref="#PWR?"  Part="1"
-AR Path="/5FD6EE9C/6118ACE0/627F4FF5" Ref="#PWR?"  Part="1"
-F 0 "#PWR?" H 4300 4650 50  0001 C CNN
+AR Path="/5FD6EE9C/6118ACE0/627F4FF5" Ref="#PWR01188"  Part="1"
+F 0 "#PWR01188" H 4300 4650 50  0001 C CNN
 F 1 "GND" H 4150 4850 50  0000 C CNN
 F 2 "" H 4300 4900 50  0001 C CNN
@@
 AR Path="/5F396002/628045F0" Ref="U?"  Part="1"
 AR Path="/5FD6F26B/628045F0" Ref="U?"  Part="1"
-AR Path="/5FD6EE9C/6118ACE0/628045F0" Ref="U?"  Part="1"
-F 0 "U?" H 4400 7050 50  0000 C CNN
+AR Path="/5FD6EE9C/6118ACE0/628045F0" Ref="U411"  Part="1"
+F 0 "U411" H 4400 7050 50  0000 C CNN
 F 1 "CD74HC283M96" H 4650 6950 50  0000 C CNN
 F 2 "Package_SO:SOIC-16_3.9x9.9mm_P1.27mm" H 4300 6300 50  0001 C CNN
@@
 AR Path="/5F396002/628045F6" Ref="#PWR?"  Part="1"
 AR Path="/5FD6F26B/628045F6" Ref="#PWR?"  Part="1"
-AR Path="/5FD6EE9C/6118ACE0/628045F6" Ref="#PWR?"  Part="1"
-F 0 "#PWR?" H 4300 5200 50  0001 C CNN
+AR Path="/5FD6EE9C/6118ACE0/628045F6" Ref="#PWR01189"  Part="1"
+F 0 "#PWR01189" H 4300 5200 50  0001 C CNN
 F 1 "+5V" H 4150 5400 50  0000 C CNN
 F 2 "" H 4300 5350 50  0001 C CNN
@@
 AR Path="/5F396002/628045FE" Ref="#PWR?"  Part="1"
 AR Path="/5FD6F26B/628045FE" Ref="#PWR?"  Part="1"
-AR Path="/5FD6EE9C/6118ACE0/628045FE" Ref="#PWR?"  Part="1"
-F 0 "#PWR?" H 4600 5150 50  0001 C CNN
+AR Path="/5FD6EE9C/6118ACE0/628045FE" Ref="#PWR01195"  Part="1"
+F 0 "#PWR01195" H 4600 5150 50  0001 C CNN
 F 1 "GND" V 4605 5272 50  0000 R CNN
 F 2 "" H 4600 5400 50  0001 C CNN
@@
 AR Path="/5F396002/62804604" Ref="C?"  Part="1"
 AR Path="/5FD6F26B/62804604" Ref="C?"  Part="1"
-AR Path="/5FD6EE9C/6118ACE0/62804604" Ref="C?"  Part="1"
-F 0 "C?" V 4221 5400 50  0000 C CNN
+AR Path="/5FD6EE9C/6118ACE0/62804604" Ref="C423"  Part="1"
+F 0 "C423" V 4221 5400 50  0000 C CNN
 F 1 "0u1" V 4312 5400 50  0000 C CNN
 F 2 "NoRef_Footprints:C_0603_1608Metric_NoRef" H 4450 5400 50  0001 C CNN
@@
 AR Path="/5F396002/6280460D" Ref="#PWR?"  Part="1"
 AR Path="/5FD6F26B/6280460D" Ref="#PWR?"  Part="1"
-AR Path="/5FD6EE9C/6118ACE0/6280460D" Ref="#PWR?"  Part="1"
-F 0 "#PWR?" H 4300 6900 50  0001 C CNN
+AR Path="/5FD6EE9C/6118ACE0/6280460D" Ref="#PWR01190"  Part="1"
+F 0 "#PWR01190" H 4300 6900 50  0001 C CNN
 F 1 "GND" H 4150 7100 50  0000 C CNN
 F 2 "" H 4300 7150 50  0001 C CNN
@@
 AR Path="/5F396002/6280462E" Ref="U?"  Part="1"
 AR Path="/5FD6F26B/6280462E" Ref="U?"  Part="1"
-AR Path="/5FD6EE9C/6118ACE0/6280462E" Ref="U?"  Part="1"
-F 0 "U?" H 4400 9300 50  0000 C CNN
+AR Path="/5FD6EE9C/6118ACE0/6280462E" Ref="U412"  Part="1"
+F 0 "U412" H 4400 9300 50  0000 C CNN
 F 1 "CD74HC283M96" H 4650 9200 50  0000 C CNN
 F 2 "Package_SO:SOIC-16_3.9x9.9mm_P1.27mm" H 4300 8550 50  0001 C CNN
@@
 AR Path="/5F396002/62804634" Ref="#PWR?"  Part="1"
 AR Path="/5FD6F26B/62804634" Ref="#PWR?"  Part="1"
-AR Path="/5FD6EE9C/6118ACE0/62804634" Ref="#PWR?"  Part="1"
-F 0 "#PWR?" H 4300 7450 50  0001 C CNN
+AR Path="/5FD6EE9C/6118ACE0/62804634" Ref="#PWR01191"  Part="1"
+F 0 "#PWR01191" H 4300 7450 50  0001 C CNN
 F 1 "+5V" H 4150 7650 50  0000 C CNN
 F 2 "" H 4300 7600 50  0001 C CNN
@@
 AR Path="/5F396002/6280463C" Ref="#PWR?"  Part="1"
 AR Path="/5FD6F26B/6280463C" Ref="#PWR?"  Part="1"
-AR Path="/5FD6EE9C/6118ACE0/6280463C" Ref="#PWR?"  Part="1"
-F 0 "#PWR?" H 4600 7400 50  0001 C CNN
+AR Path="/5FD6EE9C/6118ACE0/6280463C" Ref="#PWR01196"  Part="1"
+F 0 "#PWR01196" H 4600 7400 50  0001 C CNN
 F 1 "GND" V 4605 7522 50  0000 R CNN
 F 2 "" H 4600 7650 50  0001 C CNN
@@
 AR Path="/5F396002/62804642" Ref="C?"  Part="1"
 AR Path="/5FD6F26B/62804642" Ref="C?"  Part="1"
-AR Path="/5FD6EE9C/6118ACE0/62804642" Ref="C?"  Part="1"
-F 0 "C?" V 4221 7650 50  0000 C CNN
+AR Path="/5FD6EE9C/6118ACE0/62804642" Ref="C424"  Part="1"
+F 0 "C424" V 4221 7650 50  0000 C CNN
 F 1 "0u1" V 4312 7650 50  0000 C CNN
 F 2 "NoRef_Footprints:C_0603_1608Metric_NoRef" H 4450 7650 50  0001 C CNN
@@
 AR Path="/5F396002/6280464B" Ref="#PWR?"  Part="1"
 AR Path="/5FD6F26B/6280464B" Ref="#PWR?"  Part="1"
-AR Path="/5FD6EE9C/6118ACE0/6280464B" Ref="#PWR?"  Part="1"
-F 0 "#PWR?" H 4300 9150 50  0001 C CNN
+AR Path="/5FD6EE9C/6118ACE0/6280464B" Ref="#PWR01192"  Part="1"
+F 0 "#PWR01192" H 4300 9150 50  0001 C CNN
 F 1 "GND" H 4305 9227 50  0000 C CNN
 F 2 "" H 4300 9400 50  0001 C CNN
@@
 AR Path="/5F396002/62824AAC" Ref="#PWR?"  Part="1"
 AR Path="/5FD6F26B/62824AAC" Ref="#PWR?"  Part="1"
-AR Path="/5FD6EE9C/6118ACE0/62824AAC" Ref="#PWR?"  Part="1"
-F 0 "#PWR?" H 3750 1050 50  0001 C CNN
+AR Path="/5FD6EE9C/6118ACE0/62824AAC" Ref="#PWR01158"  Part="1"
+F 0 "#PWR01158" H 3750 1050 50  0001 C CNN
 F 1 "GND" V 3755 1172 50  0000 R CNN
 F 2 "" H 3750 1300 50  0001 C CNN
@@
 AR Path="/5F396002/628398D6" Ref="#PWR?"  Part="1"
 AR Path="/5FD6F26B/628398D6" Ref="#PWR?"  Part="1"
-AR Path="/5FD6EE9C/6118ACE0/628398D6" Ref="#PWR?"  Part="1"
-F 0 "#PWR?" H 3750 8800 50  0001 C CNN
+AR Path="/5FD6EE9C/6118ACE0/628398D6" Ref="#PWR01173"  Part="1"
+F 0 "#PWR01173" H 3750 8800 50  0001 C CNN
 F 1 "GND" H 3755 8877 50  0000 C CNN
 F 2 "" H 3750 9050 50  0001 C CNN
@@
 AR Path="/5F396002/6283C7E0" Ref="#PWR?"  Part="1"
 AR Path="/5FD6F26B/6283C7E0" Ref="#PWR?"  Part="1"
-AR Path="/5FD6EE9C/6118ACE0/6283C7E0" Ref="#PWR?"  Part="1"
-F 0 "#PWR?" H 3750 8300 50  0001 C CNN
+AR Path="/5FD6EE9C/6118ACE0/6283C7E0" Ref="#PWR01159"  Part="1"
+F 0 "#PWR01159" H 3750 8300 50  0001 C CNN
 F 1 "GND" H 3755 8377 50  0000 C CNN
 F 2 "" H 3750 8550 50  0001 C CNN
