File: ECAD/psMCU/KiCad/LogicOR.sch (KiCad schematic (older format))
At the start: 10 parts, among them U137 SN74HC32PW, U138 SN74HC32PW, U139 SN74HC245PW, U140 SN74LVC1G04DCK, U141 SN74LVC1G126DCK

Commit message: Sch: Cleanup + Small fixes
Parts:
- added C504: 10u, symbol Device:CP_Small
Connections:
- wire segments 103 -> 105
Changed lines of the file:
@@
 $Descr A4 11693 8268
 encoding utf-8
-Sheet 74 109
+Sheet 6 109
 Title "psMCU"
 Date "2022-02-13"
@@
 AR Path="/5FF66C9F/600C00E8/60419344" Ref="#PWR0636"  Part="1"
 F 0 "#PWR0636" H 6150 600 50  0001 C CNN
-F 1 "+5V" H 6000 850 50  0000 C CNN
+F 1 "+5V" H 6092 787 50  0000 R CNN
 F 2 "" H 6150 750 50  0001 C CNN
 F 3 "" H 6150 750 50  0001 C CNN
@@
 Entry Wire Line
 	6900 1250 7000 1350
+$Comp
+L Device:CP_Small C?
+U 1 1 6597E073
+P 7450 900
+AR Path="/62043340/6597E073" Ref="C?"  Part="1"
+AR Path="/5FD6B215/6597E073" Ref="C?"  Part="1"
+AR Path="/5FF66C9F/600BE39A/6597E073" Ref="C?"  Part="1"
+AR Path="/5FF66C9F/600C00E8/6597E073" Ref="C504"  Part="1"
+F 0 "C504" H 7538 946 50  0000 L CNN
+F 1 "10u" H 7538 855 50  0000 L CNN
+F 2 "" H 7450 900 50  0001 C CNN
+F 3 "~" H 7450 900 50  0001 C CNN
+	1    7450 900
+	1    0    0    -1
+$EndComp
+$Comp
+L power:GND #PWR?
+U 1 1 6597E079
+P 7450 1050
+AR Path="/6597E079" Ref="#PWR?"  Part="1"
+AR Path="/62043340/6597E079" Ref="#PWR?"  Part="1"
+AR Path="/5FD6B215/6597E079" Ref="#PWR?"  Part="1"
+AR Path="/5FF66C9F/600BE39A/6597E079" Ref="#PWR?"  Part="1"
+AR Path="/5FF66C9F/600C00E8/6597E079" Ref="#PWR07"  Part="1"
+F 0 "#PWR07" H 7450 800 50  0001 C CNN
+F 1 "GND" H 7455 877 50  0000 C CNN
+F 2 "" H 7450 1050 50  0001 C CNN
+F 3 "" H 7450 1050 50  0001 C CNN
+	1    7450 1050
+	1    0    0    -1
+$EndComp
+Wire Wire Line
+	7450 1050 7450 1000
+Wire Wire Line
+	7450 750  7450 800
+$Comp
+L power:+5V #PWR?
+U 1 1 6597E081
+P 7450 750
+AR Path="/6597E081" Ref="#PWR?"  Part="1"
+AR Path="/62043340/6597E081" Ref="#PWR?"  Part="1"
+AR Path="/5FD6B215/6597E081" Ref="#PWR?"  Part="1"
+AR Path="/5FF66C9F/600BE39A/6597E081" Ref="#PWR?"  Part="1"
+AR Path="/5FF66C9F/600C00E8/6597E081" Ref="#PWR02"  Part="1"
+F 0 "#PWR02" H 7450 600 50  0001 C CNN
+F 1 "+5V" H 7465 923 50  0000 C CNN
+F 2 "" H 7450 750 50  0001 C CNN
+F 3 "" H 7450 750 50  0001 C CNN
+	1    7450 750
+	1    0    0    -1
+$EndComp
 Wire Bus Line
 	1400 900  1400 1600
