File: ECAD/RemoteCtrl/KiCad/RemoteCtrl.sch (KiCad schematic (older format))
At the start: 19 parts, among them J1 UI

Commit message: Remote control work.
Connections:
- net +5V: now also R8.2
- net GND: no longer R8.2
Changed lines of the file:
@@
 Wire Wire Line
 	4000 2600 4000 2700
-$Comp
-L power:GND #PWR?
-U 1 1 6102C7A0
-P 4000 2700
-AR Path="/60F73904/6102C7A0" Ref="#PWR?"  Part="1"
-AR Path="/60FA12D6/6102C7A0" Ref="#PWR?"  Part="1"
-AR Path="/60FA686E/6102C7A0" Ref="#PWR?"  Part="1"
-AR Path="/60FA7824/6102C7A0" Ref="#PWR?"  Part="1"
-AR Path="/60FA8167/6102C7A0" Ref="#PWR?"  Part="1"
-AR Path="/60FA8857/6102C7A0" Ref="#PWR?"  Part="1"
-AR Path="/60FAB88D/6102C7A0" Ref="#PWR?"  Part="1"
-AR Path="/60FAB893/6102C7A0" Ref="#PWR?"  Part="1"
-AR Path="/6102C7A0" Ref="#PWR0108"  Part="1"
-F 0 "#PWR0108" H 4000 2450 50  0001 C CNN
-F 1 "GND" H 4005 2527 50  0000 C CNN
-F 2 "" H 4000 2700 50  0001 C CNN
-F 3 "" H 4000 2700 50  0001 C CNN
-	1    4000 2700
-	-1   0    0    -1
-$EndComp
 Wire Wire Line
 	3550 2300 3350 2300
@@
 	1    0    0    -1
 $EndComp
+$Comp
+L power:+5V #PWR?
+U 1 1 60A16264
+P 4000 2700
+F 0 "#PWR?" H 4000 2550 50  0001 C CNN
+F 1 "+5V" H 4015 2873 50  0000 C CNN
+F 2 "" H 4000 2700 50  0001 C CNN
+F 3 "" H 4000 2700 50  0001 C CNN
+	1    4000 2700
+	-1   0    0    1
+$EndComp
 $EndSCHEMATC

Commit message: Finished RemoteCtrl pcb
Parts:
- D1, D10, D11, D2, D7, D8, D9: footprint LED_THT:LED_D3.0mm -> LED_THT:LED_D5.0mm
Changed lines of the file:
@@
 Title "Remote Control"
 Date "2021-03-30"
-Rev "v0.1"
+Rev "v1.0"
 Comp "Philipp Schilk"
 Comment1 ""
@@
 F 0 "D11" H 5293 2995 50  0000 C CNN
 F 1 "LED" H 5293 3086 50  0000 C CNN
-F 2 "LED_THT:LED_D3.0mm" H 5300 3250 50  0001 C CNN
+F 2 "LED_THT:LED_D5.0mm" H 5300 3250 50  0001 C CNN
 F 3 "~" H 5300 3250 50  0001 C CNN
 	1    5300 3250
@@
 F 0 "D10" H 5293 2045 50  0000 C CNN
 F 1 "LED" H 5293 2136 50  0000 C CNN
-F 2 "LED_THT:LED_D3.0mm" H 5300 2300 50  0001 C CNN
+F 2 "LED_THT:LED_D5.0mm" H 5300 2300 50  0001 C CNN
 F 3 "~" H 5300 2300 50  0001 C CNN
 	1    5300 2300
@@
 F 0 "D9" H 5293 1095 50  0000 C CNN
 F 1 "LED" H 5293 1186 50  0000 C CNN
-F 2 "LED_THT:LED_D3.0mm" H 5300 1350 50  0001 C CNN
+F 2 "LED_THT:LED_D5.0mm" H 5300 1350 50  0001 C CNN
 F 3 "~" H 5300 1350 50  0001 C CNN
 	1    5300 1350
@@
 F 0 "D8" H 3693 2517 50  0000 C CNN
 F 1 "LED" H 3693 2426 50  0000 C CNN
-F 2 "LED_THT:LED_D3.0mm" H 3700 2300 50  0001 C CNN
+F 2 "LED_THT:LED_D5.0mm" H 3700 2300 50  0001 C CNN
 F 3 "~" H 3700 2300 50  0001 C CNN
 	1    3700 2300
@@
 F 0 "D7" H 3693 1095 50  0000 C CNN
 F 1 "LED" H 3693 1186 50  0000 C CNN
-F 2 "LED_THT:LED_D3.0mm" H 3700 1350 50  0001 C CNN
+F 2 "LED_THT:LED_D5.0mm" H 3700 1350 50  0001 C CNN
 F 3 "~" H 3700 1350 50  0001 C CNN
 	1    3700 1350
@@
 F 0 "D2" H 2093 2045 50  0000 C CNN
 F 1 "LED" H 2093 2136 50  0000 C CNN
-F 2 "LED_THT:LED_D3.0mm" H 2100 2300 50  0001 C CNN
+F 2 "LED_THT:LED_D5.0mm" H 2100 2300 50  0001 C CNN
 F 3 "~" H 2100 2300 50  0001 C CNN
 	1    2100 2300
@@
 F 0 "D1" H 2093 1095 50  0000 C CNN
 F 1 "LED" H 2093 1186 50  0000 C CNN
-F 2 "LED_THT:LED_D3.0mm" H 2100 1350 50  0001 C CNN
+F 2 "LED_THT:LED_D5.0mm" H 2100 1350 50  0001 C CNN
 F 3 "~" H 2100 1350 50  0001 C CNN
 	1    2100 1350
